Commit message: successful

File: my_robot/urdf/my_robot.xacro (robot description, xacro)
@@ -27,6 +27,6 @@
 		<box size=".4 .2 .1"/>
 	  </geometry>
-	  <material name="blue">
-		<color rgba="0 0 1 1"/>
+	  <material name="yellow">
+		<color rgba="1 1 0 1"/>
 	  </material>
 	</visual>
@@ -87,6 +87,6 @@
 	<cylinder radius="0.1" length="0.05"/>
 	  </geometry>
-	  <material name="green">
-		<color rgba="0 1 0 1"/>
+	  <material name="orange">
+		<color rgba="1 0.5 0 1"/>
 	  </material>
 	</visual>
@@ -115,6 +115,6 @@
 	<cylinder radius="0.1" length="0.05"/>
 	  </geometry>
-	 <material name="green">
-		<color rgba="0 1 0 1"/>
+	 <material name="orange">
+		<color rgba="1 0.5 0 1"/>
 	  </material>
 	</visual>
@@ -211,11 +211,11 @@
   <!-- ============ GAZEBO MATERIALS ============ -->
   <gazebo reference="chassis">
-    <material>Gazebo/Blue</material>
+    <material>Gazebo/Yellow</material>
   </gazebo>
   <gazebo reference="left_wheel">
-    <material>Gazebo/Green</material>
+    <material>Gazebo/Orange</material>
   </gazebo>
   <gazebo reference="right_wheel">
-    <material>Gazebo/Green</material>
+    <material>Gazebo/Orange</material>
   </gazebo>
   <gazebo reference="camera">

Commit message: dimension and radius change

File: my_robot/urdf/my_robot.xacro (robot description, xacro)
@@ -19,5 +19,5 @@
 	  <origin xyz="0 0 0" rpy=" 0 0 0"/>
 	  <geometry>
-		<box size=".4 .2 .1"/>
+		<box size=".4 .1 .1"/>
 	  </geometry>
 	</collision>
@@ -25,5 +25,5 @@
 	  <origin xyz="0 0 0" rpy=" 0 0 0"/>
 	  <geometry>
-		<box size=".4 .2 .1"/>
+		<box size=".4 .1 .1"/>
 	  </geometry>
 	  <material name="yellow">
@@ -78,5 +78,5 @@
 	  <origin xyz="0 0 0" rpy="0 1.5707 1.5707"/>
 	  <geometry>
-	<cylinder radius="0.1" length="0.05"/>
+	<cylinder radius="0.05" length="0.05"/>
 	  </geometry>
 	</collision>
@@ -85,5 +85,5 @@
 	  <origin xyz="0 0 0" rpy="0 1.5707 1.5707"/>
 	  <geometry>
-	<cylinder radius="0.1" length="0.05"/>
+	<cylinder radius="0.05" length="0.05"/>
 	  </geometry>
 	  <material name="orange">
@@ -106,5 +106,5 @@
 	  <origin xyz="0 0 0" rpy="0 1.5707 1.5707"/>
 	  <geometry>
-	<cylinder radius="0.1" length="0.05"/>
+	<cylinder radius="0.05" length="0.05"/>
 	  </geometry>
 	</collision>
@@ -113,5 +113,5 @@
 	  <origin xyz="0 0 0" rpy="0 1.5707 1.5707"/>
 	  <geometry>
-	<cylinder radius="0.1" length="0.05"/>
+	<cylinder radius="0.05" length="0.05"/>
 	  </geometry>
 	 <material name="orange">
@@ -181,5 +181,5 @@
 	<!-- Left wheel joint -->
 	<joint type="continuous" name="left_wheel_hinge">
-		<origin xyz="0 0.15 0" rpy="0 0 0"/>
+		<origin xyz="0 0.06 -0.05" rpy="0 0 0"/>
 		<child link="left_wheel"/>
 		<parent link="chassis"/>
@@ -190,5 +190,5 @@
 	<!-- Right wheel joint -->
 	  <joint type="continuous" name="right_wheel_hinge">
-		<origin xyz="0 -0.15 0" rpy="0 0 0"/>
+		<origin xyz="0 -0.06 -0.05" rpy="0 0 0"/>
 		<child link="right_wheel"/>
 		<parent link="chassis"/>
